File: main.sch (EAGLE design)
At the start: 11 parts

Commit message: modules advancement
Parts:
- removed U$1, U$2, U$3: 2X20_FEMALE_HEADER_PINV1, SamuelLibrary:2X20_FEMALE_HEADER_PINV1
- added DIO0, DIO1, DIO2, DIO3, DIO4, DIO5, DIO6, DIO7: 3X1_MALE_HEADER_PIN, SamuelLibrary:3X1_MALE_HEADER_PIN
- added GPIO: 2X20_FEMALE_HEADER_PINV1, SamuelLibrary:2X20_FEMALE_HEADER_PINV1
- added I2C: 4X1_MALE_HEADER_PIN4X1_MALE_HEADER_PIN, SamuelLibrary:4X1_MALE_HEADER_PIN4X1_MALE_HEADER_PIN
- added R1, R2, R3, R6, R7, R8: 1-2176053-4, Resistors:1-2176053-4
- added R11: 20, rcl:R-EU_R0603
- added R12: 604k, rcl:R-EU_R0603
- added U$4: MCP2515-QFN, SamuelLibrary:MCP2515-QFN
- R4: value 20 -> 1-2176053-4; device rcl:R-EU_R0603 -> Resistors:1-2176053-4
- R5: value 604k -> 1-2176053-4; device rcl:R-EU_R0603 -> Resistors:1-2176053-4
Connections:
- removed net VIN: BUCK1.IN, C1.1, C2.1, R5.2
- new net 3.3V: GPIO.2
- new net 5V: DIO0.2, DIO1.2, DIO2.2, DIO3.2, DIO4.2, DIO5.2, DIO6.2, DIO7.2, GPIO.1, GPIO.3
- new net N$10: GPIO.11
- new net N$12: GPIO.15
- new net N$13: GPIO.17
- new net N$15: GPIO.21
- new net N$16: GPIO.23
- new net N$17: GPIO.25
- new net N$18: DIO4.1, R5.1
- new net N$19: DIO6.1, R7.1
- new net N$20: GPIO.31
- new net N$22: GPIO.35
- new net N$23: GPIO.37
- new net N$24: GPIO.39
- new net N$26: DIO7.1, R8.1
- new net N$28: GPIO.8
- new net N$29: GPIO.10
- new net N$30: GPIO.12
- new net N$31: GPIO.14
- new net N$32: GPIO.16
- new net N$33: GPIO.18
- new net N$34: GPIO.20
- new net N$35: GPIO.22
- new net N$36: GPIO.24
- new net N$37: DIO5.1, R6.1
- new net N$39: GPIO.30
- new net N$40: GPIO.32
- new net N$41: GPIO.34
- new net N$42: GPIO.36
- new net N$43: GPIO.38
- new net N$44: DIO3.1, R4.1
- new net N$46: DIO1.1, R2.1
- new net N$5: DIO0.1, R1.1
- new net N$7: DIO2.1, R3.1
- new net N$8: GPIO.7
- new net N$9: GPIO.9
- new net SCL: GPIO.6
- new net SDA: GPIO.4
- new net VBATT+: BUCK1.IN, C1.1, C2.1, R12.2
- net EN: now also R12.1; no longer R5.1
- net GND: now also DIO0.3, DIO1.3, DIO2.3, DIO3.3, DIO4.3, DIO5.3, DIO6.3, DIO7.3, GPIO.13, GPIO.19, GPIO.26, GPIO.29, GPIO.33, GPIO.40, GPIO.5
- net N$1: now also R11.2; no longer R4.2
- net N$3: now also R11.1; no longer R4.1
Other:
- moved on the sheet: BUCK1, C1, C2, C3, C4, C7

Commit message: peripherals advancement
Parts:
- added PWM0, PWM1: 3X1_MALE_HEADER_PIN, SamuelLibrary:3X1_MALE_HEADER_PIN
- added R10, R13, R14, R15, R16, R17, R18, R19, R20, R9: 20k, Resistors:1-2176053-4
- added R23: 20, rcl:R-EU_R0603
- added R24: 604k, rcl:R-EU_R0603
- R1, R2, R3, R4, R5, R6, R7, R8: value 1-2176053-4 -> 20k
- R11: value 20 -> 20k; device rcl:R-EU_R0603 -> Resistors:1-2176053-4
- R12: value 604k -> 20k; device rcl:R-EU_R0603 -> Resistors:1-2176053-4
Connections:
- net 5V renamed +5V
- removed net 3.3V: GPIO.2
- removed net N$20: GPIO.31
- removed net N$41: GPIO.34
- new net +3V3: GPIO.2, I2C.3, R1.2, R11.2, R13.2, R15.2, R3.2, R5.2, R7.2, R9.2
- new net 6V: PWM0.2, PWM1.2
- new net N$11: R3.1, R4.2
- new net N$14: R5.1, R6.2
- new net N$21: R7.1, R8.2
- new net N$25: R10.2, R9.1
- new net N$27: R11.1, R12.2
- new net N$38: R13.1, R14.2
- new net N$45: R15.1, R16.2
- new net N$47: R17.1, R18.2
- new net N$49: R19.1, R20.2
- new net N$6: R1.1, R2.2
- new net PWM0: GPIO.31, PWM0.1, R17.2
- new net PWM1: GPIO.34, PWM1.1, R19.2
- net EN: now also R24.1; no longer R12.1
- net GND: now also I2C.4, PWM0.3, PWM1.3, R18.1, R20.1
- net N$1: now also R23.2; no longer R11.2
- net N$18: now also R10.1; no longer R5.1
- net N$19: now also R14.1; no longer R7.1
- net N$26: now also R16.1; no longer R8.1
- net N$3: now also R23.1; no longer R11.1
- net N$37: now also R12.1; no longer R6.1
- net N$44: now also R8.1; no longer R4.1
- net N$46: now also R4.1; no longer R2.1
- net N$5: now also R2.1; no longer R1.1
- net N$7: now also R6.1; no longer R3.1
- net SCL: now also I2C.2
- net SDA: now also I2C.1
- net VBATT+: now also R24.2; no longer R12.2
Other:
- note added: "AI"
- note added: "CAN"
- note added: "DIO"
- note added: "GPIO"
- note added: "I2C"
- note added: "PWM"
- moved on the sheet: DIO0, DIO1, DIO2, DIO3, DIO4, DIO5, DIO6, DIO7, I2C, R1, R2, R3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
