File: main.sch (EAGLE design)
At the start: 78 parts, among them M1 MOSFET

Commit message: dope pwr led system
Parts:
- removed PWR: (no value), SamuelLibrary:WL-SMCC_0603_R_V_Y_150060VS73220
- added D1, D10, D2, D3, D4, D5, D6, D7, D8, D9: (no value), SamuelLibrary:WL-SMCD_0603_150060VS55040
- added M2: MOSFET, SamuelLibrary:MOSFET
- added R33, R34, R35, R36: 49.9, SamuelLibrary:0603_RESISTOR
- added R37: 10k, SamuelLibrary:1206_RESISTOR
- added R38: 120, SamuelLibrary:0603_RESISTOR
- R1: value 300k -> (none); device SamuelLibrary:2512_RESISTOR -> SamuelLibrary:0603_RESISTOR
- R32: value 165 -> 49.9; device SamuelLibrary:0805_RESISTOR -> SamuelLibrary:0603_RESISTOR
Connections:
- removed net 6V: PWM0.2, PWM1.2
- removed net N$42: GPIO.36
- removed net N$54: PWR.+, R31.P$2
- new net N$18: D7.+, R35.P$2
- new net N$19: D10.+, D9._
- new net N$23: M2.P$3, R37.P$2, R38.P$1
- new net N$24: D10._, D2._, D4._, D6._, D8._, M2.P$1
- new net N$5: D1._, D2.+
- new net N$7: D1.+, R32.P$2
- net +5V: now also PWM0.2, PWM1.2, R32.P$1, R33.P$1, R34.P$1, R35.P$1, R36.P$1
- net COMM_GRN: now also GPIO.36; no longer GPIO.37
- net DIO0: now also GPIO.39
- net DIO1: now also GPIO.37
- net DIO2: now also GPIO.35
- net DIO3: now also GPIO.17
- net DIO4: now also GPIO.15
- net DIO5: now also GPIO.11
- net DIO6: now also GPIO.9
- net DIO7: now also GPIO.7
- net GND: now also M2.P$2, R31.P$1, R37.P$1; no longer PWR.-, R32.P$1
- net N$10: now also D5._, D6.+; no longer GPIO.11
- net N$12: now also D5.+, R34.P$2; no longer GPIO.15
- net N$13: now also D7._, D8.+; no longer GPIO.17
- net N$22: now also D9.+, R36.P$2; no longer GPIO.35
- net N$56: now also R31.P$2; no longer R32.P$2
- net N$8: now also D3._, D4.+; no longer GPIO.7
- net N$9: now also D3.+, R33.P$2; no longer GPIO.9
- net PWR: now also R38.P$2; no longer GPIO.39, R31.P$1
- net SPI_MISO: now also GPIO.22; no longer GPIO.20
- net SPI_MOSI: now also GPIO.20; no longer GPIO.22
Other:
- moved on the sheet: COMM, I2C, M1, R28, R29, R30, R31, R32, RSL

Commit message: dope led system led placement
Parts:
- renumbered ADC124S051 to ADC124, LP2590 to LP2950
Connections:
- removed net N$28: GPIO.8
- removed net N$29: GPIO.10
- removed net N$30: GPIO.12
- removed net N$31: GPIO.14
- removed net N$32: GPIO.16
- removed net N$39: GPIO.30
- net +5V: now also R32.P$2, R33.P$2, R34.P$2, R35.P$2, R36.P$2; no longer R32.P$1, R33.P$1, R34.P$1, R35.P$1, R36.P$1
- net AN_CS: now also GPIO.8
- net AN_DIN: now also GPIO.14
- net AN_DOUT: now also GPIO.12
- net AN_SCLK: now also GPIO.10
- net N$12: now also R34.P$1; no longer R34.P$2
- net N$18: now also R35.P$1; no longer R35.P$2
- net N$22: now also R36.P$1; no longer R36.P$2
- net N$7: now also R32.P$1; no longer R32.P$2
- net N$9: now also R33.P$1; no longer R33.P$2
- net PWR: now also GPIO.30
- net RSL: now also GPIO.16
Other:
- moved on the sheet: D1, D10, D2, D3, D4, D5, D6, D7, D8, D9, R32, R33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

Commit message: board layout and planes
Parts:
- VIN: value 2X1_MALE_HEADER_PIN -> CTF020V8; device SamuelLibrary:2X1_MALE_HEADER_PIN -> SamuelLibrary:CTF020V8
Changed lines of the file:
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@@
 <part name="M1" library="SamuelLibrary" deviceset="MOSFET" device="" package3d_urn="urn:adsk.eagle:package:29090892/1"/>
 <part name="SUPPLY39" library="supply2" library_urn="urn:adsk.eagle:library:372" deviceset="GND" device=""/>
-<part name="VIN" library="SamuelLibrary" deviceset="2X1_MALE_HEADER_PIN" device="" package3d_urn="urn:adsk.eagle:package:29048268/1"/>
 <part name="SUPPLY41" library="supply2" library_urn="urn:adsk.eagle:library:372" deviceset="GND" device=""/>
 <part name="COMM" library="SamuelLibrary" deviceset="WL-SBCC_0603" device="" package3d_urn="urn:adsk.eagle:package:19028034/3" technology="_150060RV75240"/>
@@
 <part name="R36" library="SamuelLibrary" deviceset="0603_RESISTOR" device="" package3d_urn="urn:adsk.eagle:package:28923673/1" value="49.9"/>
 <part name="P+21" library="supply1" library_urn="urn:adsk.eagle:library:371" deviceset="+5V" device=""/>
+<part name="VIN" library="SamuelLibrary" deviceset="CTF020V8" device=""/>
 </parts>
 <sheets>
@@
 <attribute name="VALUE" x="107.315" y="131.445" size="1.778" layer="96"/>
 </instance>
-<instance part="VIN" gate="G$1" x="30.48" y="203.2" smashed="yes">
-<attribute name="NAME" x="27.94" y="208.28" size="1.27" layer="95"/>
-</instance>
 <instance part="SUPPLY41" gate="GND" x="12.7" y="193.04" smashed="yes">
 <attribute name="VALUE" x="10.795" y="189.865" size="1.778" layer="96"/>
@@
 <instance part="P+21" gate="1" x="525.78" y="203.2" smashed="yes">
 <attribute name="VALUE" x="523.24" y="203.2" size="1.778" layer="96" rot="R180"/>
+</instance>
+<instance part="VIN" gate="G$1" x="30.48" y="203.2" smashed="yes">
+<attribute name="NAME" x="27.94" y="208.28" size="1.27" layer="95"/>
 </instance>
 </instances>
@@
 </segment>
 <segment>
-<pinref part="VIN" gate="G$1" pin="2"/>
 <wire x1="22.86" y1="200.66" x2="12.7" y2="200.66" width="0.1524" layer="91"/>
 <wire x1="12.7" y1="200.66" x2="12.7" y2="195.58" width="0.1524" layer="91"/>
 <pinref part="SUPPLY41" gate="GND" pin="GND"/>
+<pinref part="VIN" gate="G$1" pin="2"/>
 </segment>
 <segment>
@@
 </segment>
 <segment>
-<pinref part="VIN" gate="G$1" pin="1"/>
 <wire x1="22.86" y1="205.74" x2="12.7" y2="205.74" width="0.1524" layer="91"/>
 <label x="12.7" y="205.74" size="1.778" layer="91"/>
-</segment>
-</net>
+<pinref part="VIN" gate="G$1" pin="1"/>
+</segment>
+</net>
